Commit message: Fix F1 car Y-up export and ship a real RViz config
Regenerate GrabCAD STLs with CAD Y-up mapped to ROS Z-up so wheels sit
on the ground under the body, and point launch at an odom-framed RViz
config with RobotModel, TF, Grid, LaserScan, and Odometry.

File: eufs-f1-sim/overlay/eufs_racecar/eufs_racecar/urdf/racecar.xacro (robot description, xacro)
@@ -61,5 +61,5 @@
   </link>
   <joint name="left_rear_wheel_joint" type="continuous">
-    <origin xyz="-0.0000 0.6466 0.4313" rpy="1.5708 0 0" />
+    <origin xyz="0.0000 0.6466 0.3095" rpy="1.5708 0 0" />
     <parent link="chassis" />
     <child link="left_rear_wheel" />
@@ -82,5 +82,5 @@
   </link>
   <joint name="right_rear_wheel_joint" type="continuous">
-    <origin xyz="0.0000 -0.6466 0.4326" rpy="1.5708 0 0" />
+    <origin xyz="-0.0000 -0.6466 0.3108" rpy="1.5708 0 0" />
     <parent link="chassis" />
     <child link="right_rear_wheel" />
@@ -102,5 +102,5 @@
   </link>
   <joint name="left_steering_hinge_joint" type="revolute">
-    <origin xyz="3.2800 0.5818 0.3242" rpy="0 1.5708 0" />
+    <origin xyz="3.2800 0.5818 0.4179" rpy="0 1.5708 0" />
     <parent link="chassis" />
     <child link="left_steering_hinge" />
@@ -122,5 +122,5 @@
   </link>
   <joint name="right_steering_hinge_joint" type="continuous">
-    <origin xyz="3.2800 -0.5818 0.3242" rpy="0 1.5708 0" />
+    <origin xyz="3.2800 -0.5818 0.4179" rpy="0 1.5708 0" />
     <parent link="chassis" />
     <child link="right_steering_hinge" />
@@ -191,5 +191,5 @@
   </link>
   <joint name="hokuyo_joint" type="fixed">
-    <origin xyz="0.0 0.0 1.05" rpy="0 0 0"/>
+    <origin xyz="0.0 0.0 1.1220" rpy="0 0 0"/>
     <parent link="chassis" />
     <child link="laser" />
@@ -218,5 +218,5 @@
   </link>
   <joint name="zed_camera_joint" type="fixed">
-    <origin xyz="0.35 0 0.95" rpy="0 0 0"/>
+    <origin xyz="0.35 0 1.0220" rpy="0 0 0"/>
     <parent link="chassis"/>
     <child link="zed_camera_link"/>

Commit message: Give the 10s throttle enough torque to move the car.
The dashboard already published /eufs/cmd and /eufs/cmd_vel, but
gazebo_ros_ackermann_drive was wired through the energy gate (which
turns an 8 m/s setpoint into ~0.16 m/s from rest) and wheel joints
were limited to 10 N·m, below rolling resistance. Drive now listens
on /eufs/cmd_vel with Humble-scale PID and 8000 N·m effort.

File: eufs-f1-sim/overlay/eufs_racecar/eufs_racecar/urdf/racecar.xacro (robot description, xacro)
@@ -65,5 +65,5 @@
     <child link="left_rear_wheel" />
     <axis xyz="0 0 -1" />
-    <limit effort="10" velocity="100" />
+    <limit effort="8000" velocity="200" />
   </joint>
   <xacro:wheel_transmission name="left_rear_wheel" />
@@ -86,5 +86,5 @@
     <child link="right_rear_wheel" />
     <axis xyz="0 0 -1" />
-    <limit effort="10" velocity="100" />
+    <limit effort="8000" velocity="200" />
   </joint>
   <xacro:wheel_transmission name="right_rear_wheel" />
@@ -106,5 +106,5 @@
     <child link="left_steering_hinge" />
     <axis xyz="-1 0 0" />
-    <limit lower="-1.0" upper="1.0" effort="10" velocity="100" />
+    <limit lower="-1.0" upper="1.0" effort="8000" velocity="200" />
   </joint>
   <xacro:steering_hinge_transmission name="left_steering_hinge" />
@@ -126,5 +126,5 @@
     <child link="right_steering_hinge" />
     <axis xyz="-1 0 0" />
-    <limit lower="-1.0" upper="1.0" effort="10" velocity="100" />
+    <limit lower="-1.0" upper="1.0" effort="8000" velocity="200" />
   </joint>
   <xacro:steering_hinge_transmission name="right_steering_hinge" />
@@ -147,5 +147,5 @@
     <child link="left_front_wheel" />
     <axis xyz="0 0 -1" />
-    <limit effort="10" velocity="100" />
+    <limit effort="8000" velocity="200" />
   </joint>
   <xacro:wheel_transmission name="left_front_wheel" />
@@ -168,5 +168,5 @@
     <child link="right_front_wheel" />
     <axis xyz="0 0 -1" />
-    <limit effort="10" velocity="100"/>
+    <limit effort="8000" velocity="200"/>
   </joint>
   <xacro:wheel_transmission name="right_front_wheel" />

Commit message: Stop the 10s throttle from spinning the car in place.
Humble-demo steering PID/effort on 0.1 kg hinges, plus a continuous
right steer joint, yawed the chassis instead of driving down COTA.
RViz was glued to base_link at yaw=pi so that spin looked like reverse
while gzclient stayed at S/F after the car left. Cap steering torque,
make the right hinge revolute, look down the start straight in RViz,
and follow the eufs model in Gazebo.

File: eufs-f1-sim/overlay/eufs_racecar/eufs_racecar/urdf/racecar.xacro (robot description, xacro)
@@ -106,5 +106,5 @@
     <child link="left_steering_hinge" />
     <axis xyz="-1 0 0" />
-    <limit lower="-1.0" upper="1.0" effort="8000" velocity="200" />
+    <limit lower="-1.0" upper="1.0" effort="80" velocity="8" />
   </joint>
   <xacro:steering_hinge_transmission name="left_steering_hinge" />
@@ -121,10 +121,10 @@
     </visual>
   </link>
-  <joint name="right_steering_hinge_joint" type="continuous">
+  <joint name="right_steering_hinge_joint" type="revolute">
     <origin xyz="3.2800 -0.7495 0.3450" rpy="0 1.5708 0" />
     <parent link="chassis" />
     <child link="right_steering_hinge" />
     <axis xyz="-1 0 0" />
-    <limit lower="-1.0" upper="1.0" effort="8000" velocity="200" />
+    <limit lower="-1.0" upper="1.0" effort="80" velocity="8" />
   </joint>
   <xacro:steering_hinge_transmission name="right_steering_hinge" />
