Commit message: Add GrabCAD Mercedes STEP to URDF via Open CASCADE export
Convert Assem step.STEP with cadquery-ocp into per-link STL meshes
(chassis, wings, wheels), update racecar URDF joint origins, and
document the GrabCAD source in README.

File: eufs-f1-sim/overlay/eufs_racecar/eufs_racecar/urdf/macros.xacro (robot description, xacro)
@@ -4,22 +4,22 @@
 <xacro:macro name="chassis_inertial_params">
   <origin xyz="0.1477 0 0" rpy="0 0 0" />
-  <mass value="4.0" />
-  <inertia ixx="0.010609" ixy="0"          ixz="0"
-                          iyy="0.050409"   iyz="0"
-                                           izz="0.05865" />
+  <mass value="740.0" />
+  <inertia ixx="120.0" ixy="0"       ixz="0"
+                        iyy="450.0"  iyz="0"
+                                     izz="520.0" />
 </xacro:macro>
 <xacro:macro name="left_wheels_inertial_params">
   <origin xyz="0 0 -0.0225" rpy="0 0 0" />
-  <mass value="0.34055" />
-  <inertia ixx="0.00026046" ixy="0"          ixz="0"
-                            iyy="0.00026046" iyz="0"
-                                             izz="0.00041226" />
+  <mass value="12.0" />
+  <inertia ixx="0.35" ixy="0"     ixz="0"
+                       iyy="0.70"  iyz="0"
+                                   izz="0.35" />
 </xacro:macro>
 <xacro:macro name="right_wheels_inertial_params">
   <origin xyz="0 0 0.0225" rpy="0 0 0" />
-  <mass value="0.34055" />
-  <inertia ixx="0.00026046" ixy="0"          ixz="0"
-                            iyy="0.00026046" iyz="0"
-                                             izz="0.00041226" />
+  <mass value="12.0" />
+  <inertia ixx="0.35" ixy="0"     ixz="0"
+                       iyy="0.70"  iyz="0"
+                                   izz="0.35" />
 </xacro:macro>
 <xacro:macro name="steering_hinge_inertial_params">
@@ -42,4 +42,16 @@
   <geometry>
     <mesh filename="file://$(find eufs_racecar)/meshes/chassis.STL" />
+  </geometry>
+</xacro:macro>
+<xacro:macro name="front_wing_geometry">
+  <origin xyz="0 0 0" rpy="0 0 0" />
+  <geometry>
+    <mesh filename="file://$(find eufs_racecar)/meshes/front_wing.STL" />
+  </geometry>
+</xacro:macro>
+<xacro:macro name="rear_wing_geometry">
+  <origin xyz="0 0 0" rpy="0 0 0" />
+  <geometry>
+    <mesh filename="file://$(find eufs_racecar)/meshes/rear_wing.STL" />
   </geometry>
 </xacro:macro>
@@ -81,13 +93,13 @@
 </xacro:macro>
 <xacro:macro name="left_wheels_collision_geometry">
-  <origin xyz="0 0 -0.0225" rpy="0 0 0" />
+  <origin xyz="0 0 0" rpy="0 1.5708 0" />
   <geometry>
-    <cylinder length="0.045" radius="0.05" />
+    <cylinder length="0.40" radius="0.40" />
   </geometry>
 </xacro:macro>
 <xacro:macro name="right_wheels_collision_geometry">
-  <origin xyz="0 0 0.0225" rpy="0 0 0" />
+  <origin xyz="0 0 0" rpy="0 1.5708 0" />
   <geometry>
-    <cylinder length="0.045" radius="0.05" />
+    <cylinder length="0.40" radius="0.40" />
   </geometry>
 </xacro:macro>

File: eufs-f1-sim/overlay/eufs_racecar/eufs_racecar/urdf/racecar.xacro (robot description, xacro)
@@ -11,5 +11,5 @@
   </link>
   <joint name="base_link_joint" type="fixed">
-    <origin xyz="0 0 0.05" rpy="0 0 0" />
+    <origin xyz="0 0 0" rpy="0 0 0" />
     <parent link="base_link" />
     <child link="chassis" />
@@ -25,4 +25,26 @@
     <child link="chassis_inertia" />
   </joint>
+  <link name="front_wing">
+    <visual>
+      <xacro:front_wing_geometry />
+      <material name="black" />
+    </visual>
+  </link>
+  <joint name="front_wing_joint" type="fixed">
+    <origin xyz="0 0 0" rpy="0 0 0" />
+    <parent link="chassis" />
+    <child link="front_wing" />
+  </joint>
+  <link name="rear_wing">
+    <visual>
+      <xacro:rear_wing_geometry />
+      <material name="black" />
+    </visual>
+  </link>
+  <joint name="rear_wing_joint" type="fixed">
+    <origin xyz="0 0 0" rpy="0 0 0" />
+    <parent link="chassis" />
+    <child link="rear_wing" />
+  </joint>
   <!-- Add the left rear wheel with its joints and tranmissions -->
   <link name="left_rear_wheel">
@@ -34,10 +56,10 @@
       <material name="black" />
     </visual>
-    <collision>robot
+    <collision>
       <xacro:left_wheels_collision_geometry />
     </collision>
   </link>
   <joint name="left_rear_wheel_joint" type="continuous">
-    <origin xyz="0 0.1 0" rpy="1.5708 0 0" />
+    <origin xyz="0 0.647 0.875" rpy="1.5708 0 0" />
     <parent link="chassis" />
     <child link="left_rear_wheel" />
@@ -60,5 +82,5 @@
   </link>
   <joint name="right_rear_wheel_joint" type="continuous">
-    <origin xyz="0 -0.1 0" rpy="1.5708 0 0" />
+    <origin xyz="0 -0.647 0.877" rpy="1.5708 0 0" />
     <parent link="chassis" />
     <child link="right_rear_wheel" />
@@ -78,5 +100,5 @@
   </link>
   <joint name="left_steering_hinge_joint" type="revolute">
-    <origin xyz="0.325 0.1 0" rpy="0 1.5708 0" />
+    <origin xyz="3.28 0.582 0.768" rpy="0 1.5708 0" />
     <parent link="chassis" />
     <child link="left_steering_hinge" />
@@ -96,5 +118,5 @@
   </link>
   <joint name="right_steering_hinge_joint" type="continuous">
-    <origin xyz="0.325 -0.1 0" rpy="0 1.5708 0" />
+    <origin xyz="3.28 -0.582 0.768" rpy="0 1.5708 0" />
     <parent link="chassis" />
     <child link="right_steering_hinge" />
@@ -165,5 +187,5 @@
   </link>
   <joint name="hokuyo_joint" type="fixed">
-    <origin xyz="0.265 0.0 0.075" rpy="0 0 0"/>
+    <origin xyz="0.0 0.0 1.05" rpy="0 0 0"/>
     <parent link="chassis" />
     <child link="laser" />
@@ -192,5 +214,5 @@
   </link>
   <joint name="zed_camera_joint" type="fixed">
-    <origin xyz="0.390 0 0.04" rpy="0 0 0"/>
+    <origin xyz="0.35 0 0.95" rpy="0 0 0"/>
     <parent link="chassis"/>
     <child link="zed_camera_link"/>

Commit message: Fix F1 STEP mesh grouping and launch all three GUIs on start
Regroup GrabCAD STEP solids by volume and position into chassis, wings,
and four corner wheels with centered wheel meshes and ground-aligned joints.
Restore rqt and RViz in load_car.launch.py and default container CMD.

File: eufs-f1-sim/overlay/eufs_racecar/eufs_racecar/urdf/macros.xacro (robot description, xacro)
@@ -95,5 +95,5 @@
   <origin xyz="0 0 0" rpy="0 1.5708 0" />
   <geometry>
-    <cylinder length="0.40" radius="0.40" />
+    <cylinder length="0.853" radius="0.427" />
   </geometry>
 </xacro:macro>
@@ -101,5 +101,5 @@
   <origin xyz="0 0 0" rpy="0 1.5708 0" />
   <geometry>
-    <cylinder length="0.40" radius="0.40" />
+    <cylinder length="0.853" radius="0.427" />
   </geometry>
 </xacro:macro>

File: eufs-f1-sim/overlay/eufs_racecar/eufs_racecar/urdf/racecar.xacro (robot description, xacro)
@@ -61,5 +61,5 @@
   </link>
   <joint name="left_rear_wheel_joint" type="continuous">
-    <origin xyz="0 0.647 0.875" rpy="1.5708 0 0" />
+    <origin xyz="-0.0000 0.6466 0.4313" rpy="1.5708 0 0" />
     <parent link="chassis" />
     <child link="left_rear_wheel" />
@@ -82,5 +82,5 @@
   </link>
   <joint name="right_rear_wheel_joint" type="continuous">
-    <origin xyz="0 -0.647 0.877" rpy="1.5708 0 0" />
+    <origin xyz="0.0000 -0.6466 0.4326" rpy="1.5708 0 0" />
     <parent link="chassis" />
     <child link="right_rear_wheel" />
@@ -96,9 +96,11 @@
     <visual>
       <xacro:left_steering_hinge_geometry />
-      <material name="grey" />
+      <material name="grey">
+        <color rgba="0 0 0 0" />
+      </material>
     </visual>
   </link>
   <joint name="left_steering_hinge_joint" type="revolute">
-    <origin xyz="3.28 0.582 0.768" rpy="0 1.5708 0" />
+    <origin xyz="3.2800 0.5818 0.3242" rpy="0 1.5708 0" />
     <parent link="chassis" />
     <child link="left_steering_hinge" />
@@ -114,9 +116,11 @@
     <visual>
       <xacro:right_steering_hinge_geometry />
-      <material name="grey" />
+      <material name="grey">
+        <color rgba="0 0 0 0" />
+      </material>
     </visual>
   </link>
   <joint name="right_steering_hinge_joint" type="continuous">
-    <origin xyz="3.28 -0.582 0.768" rpy="0 1.5708 0" />
+    <origin xyz="3.2800 -0.5818 0.3242" rpy="0 1.5708 0" />
     <parent link="chassis" />
     <child link="right_steering_hinge" />

Commit message: Drop leftover F1 uprights from wheel meshes and paint silver/black
The black bars poking out of the tires were Formula 1 body solids
(uprights/wishbones/brake ducts) parented onto the wheel links. Wheel
STLs are now the GrabCAD WHEEL tire+rim only. Chassis and wings use
metallic silver; tires are 0.05 black.

File: eufs-f1-sim/overlay/eufs_racecar/eufs_racecar/urdf/macros.xacro (robot description, xacro)
@@ -93,13 +93,13 @@
 </xacro:macro>
 <xacro:macro name="left_wheels_collision_geometry">
-  <origin xyz="0 0 0" rpy="0 1.5708 0" />
+  <origin xyz="0 0 0" rpy="0 0 0" />
   <geometry>
-    <cylinder length="0.853" radius="0.427" />
+    <cylinder length="0.413" radius="0.346" />
   </geometry>
 </xacro:macro>
 <xacro:macro name="right_wheels_collision_geometry">
-  <origin xyz="0 0 0" rpy="0 1.5708 0" />
+  <origin xyz="0 0 0" rpy="0 0 0" />
   <geometry>
-    <cylinder length="0.853" radius="0.427" />
+    <cylinder length="0.413" radius="0.346" />
   </geometry>
 </xacro:macro>

File: eufs-f1-sim/overlay/eufs_racecar/eufs_racecar/urdf/materials.xacro (robot description, xacro)
@@ -2,5 +2,14 @@
 <robot name="racecar" xmlns:xacro="http://www.ros.org/wiki/xacro">
 <material name="black">
-  <color rgba="0.0 0.0 0.0 1.0"/>
+  <color rgba="0.05 0.05 0.05 1.0"/>
+</material>
+<material name="tire_black">
+  <color rgba="0.05 0.05 0.05 1.0"/>
+</material>
+<material name="silver">
+  <color rgba="0.75 0.75 0.78 1.0"/>
+</material>
+<material name="rim_grey">
+  <color rgba="0.18 0.18 0.20 1.0"/>
 </material>
 <material name="blue">

File: eufs-f1-sim/overlay/eufs_racecar/eufs_racecar/urdf/racecar.xacro (robot description, xacro)
@@ -7,5 +7,5 @@
     <visual>
       <xacro:chassis_geometry/>
-      <material name="blue" />
+      <material name="silver" />
     </visual>
   </link>
@@ -28,5 +28,5 @@
     <visual>
       <xacro:front_wing_geometry />
-      <material name="black" />
+      <material name="silver" />
     </visual>
   </link>
@@ -39,5 +39,5 @@
     <visual>
       <xacro:rear_wing_geometry />
-      <material name="black" />
+      <material name="silver" />
     </visual>
   </link>
@@ -54,5 +54,5 @@
     <visual>
       <xacro:left_rear_wheel_geometry />
-      <material name="black" />
+      <material name="tire_black" />
     </visual>
     <collision>
@@ -61,5 +61,5 @@
   </link>
   <joint name="left_rear_wheel_joint" type="continuous">
-    <origin xyz="0.0000 0.6466 0.3095" rpy="1.5708 0 0" />
+    <origin xyz="0.0000 0.8221 0.3459" rpy="1.5708 0 0" />
     <parent link="chassis" />
     <child link="left_rear_wheel" />
@@ -75,5 +75,5 @@
     <visual>
       <xacro:right_rear_wheel_geometry />
-      <material name="black" />
+      <material name="tire_black" />
     </visual>
     <collision>
@@ -82,5 +82,5 @@
   </link>
   <joint name="right_rear_wheel_joint" type="continuous">
-    <origin xyz="-0.0000 -0.6466 0.3108" rpy="1.5708 0 0" />
+    <origin xyz="-0.0000 -0.8221 0.3472" rpy="1.5708 0 0" />
     <parent link="chassis" />
     <child link="right_rear_wheel" />
@@ -102,5 +102,5 @@
   </link>
   <joint name="left_steering_hinge_joint" type="revolute">
-    <origin xyz="3.2800 0.5818 0.4179" rpy="0 1.5708 0" />
+    <origin xyz="3.2800 0.7495 0.3450" rpy="0 1.5708 0" />
     <parent link="chassis" />
     <child link="left_steering_hinge" />
@@ -122,5 +122,5 @@
   </link>
   <joint name="right_steering_hinge_joint" type="continuous">
-    <origin xyz="3.2800 -0.5818 0.4179" rpy="0 1.5708 0" />
+    <origin xyz="3.2800 -0.7495 0.3450" rpy="0 1.5708 0" />
     <parent link="chassis" />
     <child link="right_steering_hinge" />
@@ -136,5 +136,5 @@
     <visual>
       <xacro:left_front_wheel_geometry />
-      <material name="black" />
+      <material name="tire_black" />
     </visual>
     <collision>
@@ -157,5 +157,5 @@
     <visual>
       <xacro:right_front_wheel_geometry />
-      <material name="black" />
+      <material name="tire_black" />
     </visual>
     <collision>
@@ -191,5 +191,5 @@
   </link>
   <joint name="hokuyo_joint" type="fixed">
-    <origin xyz="0.0 0.0 1.1220" rpy="0 0 0"/>
+    <origin xyz="0.0 0.0 1.1414" rpy="0 0 0"/>
     <parent link="chassis" />
     <child link="laser" />
@@ -214,9 +214,9 @@
         <box size="0.033 0.175 0.030"/>
       </geometry>
-      <material name="red"/>
+      <material name="grey"/>
     </visual>
   </link>
   <joint name="zed_camera_joint" type="fixed">
-    <origin xyz="0.35 0 1.0220" rpy="0 0 0"/>
+    <origin xyz="0.35 0 1.0414" rpy="0 0 0"/>
     <parent link="chassis"/>
     <child link="zed_camera_link"/>

Commit message: Paint F1 car with Classic Gazebo materials and chase RViz behind the car.
gzclient stayed white because nested SDF ambient/script blobs never bind on
STL visuals. Use EUFS-style <gazebo reference><material>NAME</material> plus
GAZEBO_MATERIAL_PATH so EUFSF1/Silver and EUFSF1/TireBlack load. RViz starts
from the stock EUFS Orbit view, Transient Local robot_description, package://
meshes, and a base_link chase camera instead of an empty odom grid.

File: eufs-f1-sim/overlay/eufs_racecar/eufs_racecar/urdf/macros.xacro (robot description, xacro)
@@ -41,5 +41,5 @@
   <origin xyz="0 0 0" rpy="0 0 0" />
   <geometry>
-    <mesh filename="file://$(find eufs_racecar)/meshes/chassis.STL" />
+    <mesh filename="package://eufs_racecar/meshes/chassis.STL" />
   </geometry>
 </xacro:macro>
@@ -47,5 +47,5 @@
   <origin xyz="0 0 0" rpy="0 0 0" />
   <geometry>
-    <mesh filename="file://$(find eufs_racecar)/meshes/front_wing.STL" />
+    <mesh filename="package://eufs_racecar/meshes/front_wing.STL" />
   </geometry>
 </xacro:macro>
@@ -53,5 +53,5 @@
   <origin xyz="0 0 0" rpy="0 0 0" />
   <geometry>
-    <mesh filename="file://$(find eufs_racecar)/meshes/rear_wing.STL" />
+    <mesh filename="package://eufs_racecar/meshes/rear_wing.STL" />
   </geometry>
 </xacro:macro>
@@ -59,5 +59,5 @@
   <origin xyz="0 0 0" rpy="0 0 0" />
   <geometry>
-    <mesh filename="file://$(find eufs_racecar)/meshes/left_rear_wheel.STL" />
+    <mesh filename="package://eufs_racecar/meshes/left_rear_wheel.STL" />
   </geometry>
 </xacro:macro>
@@ -65,5 +65,5 @@
   <origin xyz="0 0 0" rpy="0 0 0" />
   <geometry>
-    <mesh filename="file://$(find eufs_racecar)/meshes/right_rear_wheel.STL" />
+    <mesh filename="package://eufs_racecar/meshes/right_rear_wheel.STL" />
   </geometry>
 </xacro:macro>
@@ -71,5 +71,5 @@
   <origin xyz="0 0 0" rpy="0 0 0" />
   <geometry>
-    <mesh filename="file://$(find eufs_racecar)/meshes/left_front_wheel.STL" />
+    <mesh filename="package://eufs_racecar/meshes/left_front_wheel.STL" />
   </geometry>
 </xacro:macro>
@@ -77,5 +77,5 @@
   <origin xyz="0 0 0" rpy="0 0 0" />
   <geometry>
-    <mesh filename="file://$(find eufs_racecar)/meshes/right_front_wheel.STL" />
+    <mesh filename="package://eufs_racecar/meshes/right_front_wheel.STL" />
   </geometry>
 </xacro:macro>
@@ -83,5 +83,5 @@
   <origin xyz="0 0 0" rpy="0 0 0" />
   <geometry>
-    <mesh filename="file://$(find eufs_racecar)/meshes/left_steering_hinge.STL" />
+    <mesh filename="package://eufs_racecar/meshes/left_steering_hinge.STL" />
   </geometry>
 </xacro:macro>
@@ -89,5 +89,5 @@
   <origin xyz="0 0 0" rpy="0 0 0" />
   <geometry>
-    <mesh filename="file://$(find eufs_racecar)/meshes/right_steering_hinge.STL" />
+    <mesh filename="package://eufs_racecar/meshes/right_steering_hinge.STL" />
   </geometry>
 </xacro:macro>

File: eufs-f1-sim/overlay/eufs_racecar/eufs_racecar/urdf/racecar.xacro (robot description, xacro)
@@ -185,7 +185,7 @@
       <origin xyz="0 0 0" rpy="0 0 0"/>
       <geometry>
-        <mesh filename="file://$(find eufs_racecar)/meshes/hokuyo.dae"/>
-        <material name="grey" />
-      </geometry>
+        <mesh filename="package://eufs_racecar/meshes/hokuyo.dae"/>
+      </geometry>
+      <material name="grey" />
     </visual>
   </link>

Commit message: Make the car roll instead of hop, slide, and spin.
Cylinder contacts plus 1000-gain wheel torque made the chassis dance;
RViz joint_states were held at zero so the tires never turned. Use
sphere wheel collisions, a 30-gain drive PID, real Gazebo joint states,
and keep both cameras behind S/F looking down the straight.

File: eufs-f1-sim/overlay/eufs_racecar/eufs_racecar/urdf/macros.xacro (robot description, xacro)
@@ -95,5 +95,5 @@
   <origin xyz="0 0 0" rpy="0 0 0" />
   <geometry>
-    <cylinder length="0.413" radius="0.346" />
+    <sphere radius="0.346" />
   </geometry>
 </xacro:macro>
@@ -101,5 +101,5 @@
   <origin xyz="0 0 0" rpy="0 0 0" />
   <geometry>
-    <cylinder length="0.413" radius="0.346" />
+    <sphere radius="0.346" />
   </geometry>
 </xacro:macro>

File: eufs-f1-sim/overlay/eufs_racecar/eufs_racecar/urdf/racecar.xacro (robot description, xacro)
@@ -65,5 +65,5 @@
     <child link="left_rear_wheel" />
     <axis xyz="0 0 -1" />
-    <limit effort="8000" velocity="200" />
+    <limit effort="400" velocity="80" />
   </joint>
   <xacro:wheel_transmission name="left_rear_wheel" />
@@ -86,5 +86,5 @@
     <child link="right_rear_wheel" />
     <axis xyz="0 0 -1" />
-    <limit effort="8000" velocity="200" />
+    <limit effort="400" velocity="80" />
   </joint>
   <xacro:wheel_transmission name="right_rear_wheel" />
@@ -147,5 +147,5 @@
     <child link="left_front_wheel" />
     <axis xyz="0 0 -1" />
-    <limit effort="8000" velocity="200" />
+    <limit effort="400" velocity="80" />
   </joint>
   <xacro:wheel_transmission name="left_front_wheel" />
@@ -168,5 +168,5 @@
     <child link="right_front_wheel" />
     <axis xyz="0 0 -1" />
-    <limit effort="8000" velocity="200"/>
+    <limit effort="400" velocity="80"/>
   </joint>
   <xacro:wheel_transmission name="right_front_wheel" />

Commit message: Repair EUFS driving and add modular grid telemetry
Preserve corrected wheel rolling and the original single-car spawn while adding namespaced staggered grids, continuous white boundaries, managed dashboard lifecycle, and nullable telemetry tabs with graphs.

Validated with 27 focused tests, live four-car COTA and two-car stock-map spawning, 1/4/20-car geometry checks, and shutdown/restart with fresh telemetry and no stale TF warnings. Preserve deployed cone definitions in the source overlay for reproducible builds.

File: eufs-f1-sim/overlay/eufs_racecar/eufs_racecar/urdf/macros.xacro (robot description, xacro)
@@ -12,21 +12,21 @@
   <origin xyz="0 0 -0.0225" rpy="0 0 0" />
   <mass value="12.0" />
-  <inertia ixx="0.35" ixy="0"     ixz="0"
-                       iyy="0.70"  iyz="0"
-                                   izz="0.35" />
+  <inertia ixx="0.535548" ixy="0"       ixz="0"
+                       iyy="0.535548" iyz="0"
+                                   izz="0.718296" />
 </xacro:macro>
 <xacro:macro name="right_wheels_inertial_params">
   <origin xyz="0 0 0.0225" rpy="0 0 0" />
   <mass value="12.0" />
-  <inertia ixx="0.35" ixy="0"     ixz="0"
-                       iyy="0.70"  iyz="0"
-                                   izz="0.35" />
+  <inertia ixx="0.535548" ixy="0"       ixz="0"
+                       iyy="0.535548" iyz="0"
+                                   izz="0.718296" />
 </xacro:macro>
 <xacro:macro name="steering_hinge_inertial_params">
   <origin xyz="0 0 0" rpy="0 0 0" />
-  <mass value="0.100" />
-  <inertia ixx="4E-06" ixy="0"           ixz="0"
-                            iyy="4E-06"  iyz="0"
-                                              izz="4E-06" />
+  <mass value="1.0" />
+  <inertia ixx="0.005" ixy="0"       ixz="0"
+                       iyy="0.005" iyz="0"
+                                  izz="0.005" />
 </xacro:macro>
 <xacro:macro name="hokuyo_inertial_params">
@@ -39,5 +39,9 @@
 <!-- geometry macros -->
 <xacro:macro name="chassis_geometry">
-  <origin xyz="0 0 0" rpy="0 0 0" />
+  <!-- The chassis mesh is authored nose-at-negative-X, while the vehicle
+       frame places the steering/front axle at positive X (rear axle at X=0).
+       Rotate the body about Z and reflect it around the axle midpoint so the
+       visible nose follows the vehicle's forward +X direction. -->
+  <origin xyz="3.28 0 0" rpy="0 0 3.141592653589793" />
   <geometry>
     <mesh filename="package://eufs_racecar/meshes/chassis.STL" />

File: eufs-f1-sim/overlay/eufs_racecar/robots/eufs/robot.urdf.xacro (robot description, xacro)
@@ -6,4 +6,13 @@
   <xacro:arg name="forgez_E_lap" default="220.0"/>
   <xacro:arg name="forgez_R_OT" default="0.040"/>
+  <!-- Motion plant selection.  DynamicBicycle is the stock EUFS acceleration
+       plant; Ackermann is the contact-rich Gazebo velocity plant. -->
+  <xacro:arg name="vehicle_model" default="DynamicBicycle"/>
+  <xacro:arg name="command_mode" default="acceleration"/>
+  <xacro:arg name="publish_tf" default="false"/>
+  <xacro:arg name="frame_prefix" default=""/>
+  <xacro:arg name="native_remap" default="false"/>
+  <xacro:arg name="pub_ground_truth" default="true"/>
+  <xacro:arg name="noise_config" default=""/>
   <xacro:include filename="$(find eufs_racecar)/urdf/racecar.xacro"/>
   <xacro:include filename="$(find eufs_racecar)/urdf/forgez_battery.gazebo"/>
